Commit message: drivers for UR10e external control

File: ur_description/urdf/ur10e.xacro (robot description, xacro)
@@ -24,20 +24,7 @@
 <!--  Sensor-->
 <!--  <xacro:include filename="$(find realsense2_description)/urdf/test_d435i_camera.urdf.xacro" />-->
-<!--  <xacro:realsense2_camera parent="base_link" use_nominal_extrinsics="true">-->
 <!--&lt;!&ndash;    For this manual calibration, drag the gripper (tool0_controller) to the camera mass-->
 <!--        center and record here the tf values (/base_link to /tool0_controller).&ndash;&gt;-->
 <!--&lt;!&ndash;    The second rotation value (P) you should add pi constant: 2.627 = −0,515 + pi &ndash;&gt;-->
 <!--&lt;!&ndash;      <origin xyz="0.785 -0.839 0.426" rpy="-3.104 2.471 -1.613"/>&ndash;&gt;-->
-<!--      <origin xyz="0.797 -0.803 0.432" rpy="3.135 2.462 -1.577"/>-->
-<!--  </xacro:realsense2_camera>-->
-<!--  <xacro:realsense2_camera use_nominal_extrinsics="true">-->
-<!--  </xacro:realsense2_camera>-->
-  <!-- Gripper -->
-<!--  <xacro:include filename="$(find robotiq_2f_140_gripper_visualization)/urdf/robotiq_arg2f_140.xacro" />-->
-<!--  <xacro:robotiq_arg2f_140_model parent="base_link">-->
-<!--      <origin xyz="1.7 -0.833 0.424 " rpy="3.073 2.627 -1.650"/>-->
-<!--  </xacro:robotiq_arg2f_140_model>-->
-<!--&lt;!&ndash;   Gripper &ndash;&gt;-->
-<!--  <xacro:include filename="$(find robotiq_2f_140_gripper_visualization)/urdf/robotiq_arg2f_140.xacro" />-->
-<!--  <xacro:robotiq_arg2f_140_model/>-->
 </robot>
